Commit message: updated new robot model

File: udacity_bot/urdf/navbot.xacro (robot description, xacro)
@@ -3,8 +3,8 @@
     <xacro:include filename="$(find udacity_bot)/urdf/udacity_bot.gazebo" />
     <gazebo reference="left_wheel">
-      <material>Gazebo/Gray</material>
+      <material>Gazebo/Grey</material>
     </gazebo>
     <gazebo reference="right_wheel">
-      <material>Gazebo/Gray</material>
+      <material>Gazebo/Grey</material>
     </gazebo>
     <gazebo reference="chassis">
@@ -90,5 +90,5 @@
             <cylinder radius="0.1" length="0.05"/>
         </geometry>
-        <material name="gray"/>
+        <material name="grey"/>
     </visual>
   </link>
@@ -114,5 +114,5 @@
             <cylinder radius="0.1" length="0.05"/>
         </geometry>
-        <material name="gray"/>
+        <material name="grey"/>
     </visual>
   </link>
@@ -133,4 +133,33 @@
     <dynamics damping="1.0" friction="1.0"/>
   </joint>
+    <link name='top_base'>
+    <inertial>
+      <mass value="2.0"/>
+      <origin xyz="0.0 0 0" rpy=" 0 0 0"/>
+      <inertia
+          ixx="0.1" ixy="0" ixz="0"
+          iyy="0.1" iyz="0"
+          izz="0.1"
+      />
+    </inertial>
+    <collision name='top_base_collision'>
+        <origin xyz="0 0 0" rpy="0 0 0"/>
+        <geometry>
+            <box size="0.2 0.2 0.3"/>
+        </geometry>
+    </collision>
+    <visual name='top_base_visual'>
+        <origin xyz="0 0 0" rpy="0 0 0"/>
+        <geometry>
+            <box size="0.2 0.2 0.3"/>
+        </geometry>
+        <material name="green"/>
+    </visual>
+  </link>
+    <joint type="fixed" name="top_base_joint">
+        <origin xyz="0 0 0.2" rpy="0 0 0"/>
+        <child link="top_base"/>
+        <parent link="chassis"/>
+    </joint>
     <link name='camera'>
         <inertial>
@@ -160,7 +189,7 @@
     </link>
     <joint type="fixed" name="camera_joint">
-        <origin xyz="0.2 0 0" rpy="0 0 0"/>
+        <origin xyz="0 0 0.3" rpy="0 0 0"/>
         <child link="camera"/>
-        <parent link="chassis"/>
+        <parent link="top_base"/>
     </joint>
     <link name='hokuyo'>
@@ -188,36 +217,7 @@
     </link>
     <joint type="fixed" name="hokuyo_joint">
-        <origin xyz="0.15 0 0.1" rpy="0 0 0"/>
+        <origin xyz="0.15 0 0.3" rpy="0 0 0"/>
         <child link="hokuyo"/>
-        <parent link="chassis"/>
-    </joint>
-    <link name='top_base'>
-    <inertial>
-      <mass value="2.0"/>
-      <origin xyz="0.0 0 0" rpy=" 0 0 0"/>
-      <inertia
-          ixx="0.1" ixy="0" ixz="0"
-          iyy="0.1" iyz="0"
-          izz="0.1"
-      />
-    </inertial>
-    <collision name='top_base_collision'>
-        <origin xyz="0 0 0" rpy="0 0 0"/>
-        <geometry>
-            <box size="0.4 0.2 0.1"/>
-        </geometry>
-    </collision>
-    <visual name='top_base_visual'>
-        <origin xyz="0 0 0" rpy="0 0 0"/>
-        <geometry>
-            <box size="0.4 0.2 0.1"/>
-        </geometry>
-        <material name="green"/>
-    </visual>
-  </link>
-    <joint type="fixed" name="top_base_joint">
-        <origin xyz="0 0 0.1" rpy="0 0 0"/>
-        <child link="top_base"/>
-        <parent link="chassis"/>
+        <parent link="top_base"/>
     </joint>
 </robot>

Commit message: Navbot tuning and results

File: udacity_bot/urdf/navbot.xacro (robot description, xacro)
@@ -1,4 +1,4 @@
 <?xml version='1.0'?>
-<robot name="udacity_bot" xmlns:xacro="http://www.ros.org/wiki/xacro">
+<robot name="navbot" xmlns:xacro="http://www.ros.org/wiki/xacro">
     <xacro:include filename="$(find udacity_bot)/urdf/udacity_bot.gazebo" />
     <gazebo reference="left_wheel">
@@ -13,5 +13,8 @@
     <gazebo reference="top_base">
           <material>Gazebo/Green</material>
-        </gazebo>
+    </gazebo>
+    <gazebo reference="camera">
+          <material>Gazebo/RustySteel</material>
+    </gazebo>
   <link name="robot_footprint"></link>
   <joint name="robot_footprint_joint" type="fixed">
@@ -34,5 +37,5 @@
       <origin xyz="0 0 0" rpy=" 0 0 0"/>
       <geometry>
-        <box size=".4 .2 .1"/>
+        <cylinder radius="0.4" length="0.05"/>
       </geometry>
     </collision>
@@ -40,5 +43,5 @@
       <origin xyz="0 0 0" rpy=" 0 0 0"/>
       <geometry>
-        <cylinder radius="0.4" length="0.05"/>
+        <cylinder radius="0.2" length="0.05"/>
       </geometry>
       <material name="black"/>
@@ -118,5 +121,5 @@
   </link>
   <joint type="continuous" name="left_wheel_hinge">
-    <origin xyz="0 0.15 0" rpy="0 0 0"/>
+    <origin xyz="0 0.2 0" rpy="0 0 0"/>
     <child link="left_wheel"/>
     <parent link="chassis"/>
@@ -126,5 +129,5 @@
   </joint>
   <joint type="continuous" name="right_wheel_hinge">
-    <origin xyz="0 -0.15 0" rpy="0 0 0"/>
+    <origin xyz="0 -0.2 0" rpy="0 0 0"/>
     <child link="right_wheel"/>
     <parent link="chassis"/>
@@ -158,5 +161,5 @@
   </link>
     <joint type="fixed" name="top_base_joint">
-        <origin xyz="0 0 0.2" rpy="0 0 0"/>
+        <origin xyz="0 0 0.15" rpy="0 0 0"/>
         <child link="top_base"/>
         <parent link="chassis"/>
@@ -183,11 +186,9 @@
                 <box size="0.05 0.05 0.05"/>
             </geometry>
-            <material name="">
-                <color rgba="1 0 0 1"/>
-            </material>
+            <material name="steel"/>
         </visual>
     </link>
     <joint type="fixed" name="camera_joint">
-        <origin xyz="0 0 0.3" rpy="0 0 0"/>
+        <origin xyz="0.1 0 0" rpy="0 0 0"/>
         <child link="camera"/>
         <parent link="top_base"/>
@@ -217,5 +218,5 @@
     </link>
     <joint type="fixed" name="hokuyo_joint">
-        <origin xyz="0.15 0 0.3" rpy="0 0 0"/>
+        <origin xyz="0.07 0 0.185" rpy="0 0 0"/>
         <child link="hokuyo"/>
         <parent link="top_base"/>

Commit message: Finetuning and bot image added

File: udacity_bot/urdf/navbot.xacro (robot description, xacro)
@@ -121,5 +121,5 @@
   </link>
   <joint type="continuous" name="left_wheel_hinge">
-    <origin xyz="0 0.2 0" rpy="0 0 0"/>
+    <origin xyz="0 0.23 0" rpy="0 0 0"/>
     <child link="left_wheel"/>
     <parent link="chassis"/>
@@ -129,5 +129,5 @@
   </joint>
   <joint type="continuous" name="right_wheel_hinge">
-    <origin xyz="0 -0.2 0" rpy="0 0 0"/>
+    <origin xyz="0 -0.23 0" rpy="0 0 0"/>
     <child link="right_wheel"/>
     <parent link="chassis"/>

File: udacity_bot/urdf/udacity_bot.xacro (robot description, xacro)
@@ -39,5 +39,4 @@
         <box size=".4 .2 .1"/>
       </geometry>
-        <material name="blue"/>
     </visual>
     <collision name='back_caster_collision'>
